Commit message: updated launch files, urdf, and added world file and integrated the rviz

File: src/my_robot/urdf/my_robot.xacro (robot description, xacro)
@@ -1,4 +1,5 @@
 <?xml version='1.0'?>
 <robot name="my_robot" xmlns:xacro="http://www.ros.org/wiki/xacro">
+<xacro:include filename="$(find my_robot)/urdf/my_robot.gazebo" />
   <link name="robot_footprint"></link>
   <joint name="robot_footprint_joint" type="fixed">
@@ -55,3 +56,154 @@
     </visual>
   </link>
+<!-- adding Left Wheel -->
+  <link name='left_wheel'>
+    <pose>0 0 0 0 0 0</pose>
+    <inertial>
+      <mass value = "5"/>
+      <origin xyz="0 0 0" rpy=" 0 1.5707 1.5707"/>
+      <inertia
+        ixx="0.1" ixy="0" ixz="0"
+        iyy="0.1" iyz="0"
+        izz="0.1"
+      />
+    </inertial>
+    <collision name='left_wheel_collision'>
+      <origin xyz="0 0 0" rpy=" 0 1.5707 1.5707"/>
+      <geometry>
+        <!-- <cylinder>
+          <radius>0.1</radius>
+          <length>0.05</length>
+       </cylinder> -->
+       <cylinder radius="0.1" length="0.05"/>
+      </geometry>
+    </collision>
+    <visual name='left_wheel_visual'>
+      <origin xyz="0 0 0" rpy=" 0 1.5707 1.5707"/>
+      <geometry>
+        <!-- <cylinder>
+          <radius>0.1</radius>
+          <length>0.05</length>
+       </cylinder> -->
+       <cylinder radius="0.1" length="0.05"/>
+      </geometry>
+    </visual>
+  </link>
+  <joint type="continuous" name="left_wheel_hinge">
+    <origin xyz="0 0.15 0" rpy="0 0 0"/>
+    <child link="left_wheel"/>
+    <parent link="chassis"/>
+    <axis xyz="0 1 0" rpy="0 0 0"/>
+    <limit effort="10000" velocity="1000"/>
+    <dynamics damping="1.0" friction="1.0"/>
+  </joint>
+<!-- adding Right Wheel -->
+  <link name='right_wheel'>
+    <pose>0 0 0 0 0 0</pose>
+    <inertial>
+      <mass value = "5"/>
+      <origin xyz="0 0 0" rpy=" 0 1.5707 1.5707"/>
+      <inertia
+        ixx="0.1" ixy="0" ixz="0"
+        iyy="0.1" iyz="0"
+        izz="0.1"
+      />
+    </inertial>
+    <collision name='right_wheel_collision'>
+      <origin xyz="0 0 0" rpy=" 0 1.5707 1.5707"/>
+      <geometry>
+       <cylinder radius="0.1" length="0.05"/>
+      </geometry>
+    </collision>
+    <visual name='right_wheel_visual'>
+      <origin xyz="0 0 0" rpy=" 0 1.5707 1.5707"/>
+      <geometry>
+       <cylinder radius="0.1" length="0.05"/>
+      </geometry>
+    </visual>
+  </link>
+  <joint type="continuous" name="right_wheel_hinge">
+    <origin xyz="0 -0.15 0" rpy="0 0 0"/>
+    <child link="right_wheel"/>
+    <parent link="chassis"/>
+    <axis xyz="0 1 0" rpy="0 0 0"/>
+    <limit effort="10000" velocity="1000"/>
+    <dynamics damping="1.0" friction="1.0"/>
+  </joint>
+<!-- adding a Camera -->
+   <link name = 'camera'>
+    <pose>0 0 0 0 0 0</pose>
+    <inertial>
+        <mass value="0.1"/>
+        <origin xyz = "0 0 0" rpy=" 0 0 0"/>
+        <inertia
+            ixx="1e-6" ixy="0" ixz="0"
+            iyy="1e-6" iyz="0"
+            izz="1e-6"
+        />
+    </inertial>
+    <collision name='camera_collision'>
+        <origin xyz = "0 0 0" rpy=" 0 0 0"/>
+        <geometry>
+            <box size = "0.05 0.05 0.05"/>
+        </geometry>
+    </collision>
+    <visual name='camera_visual'>
+        <origin xyz = "0 0 0" rpy=" 0 0 0"/>
+        <geometry>
+            <box size = "0.05 0.05 0.05"/>
+        </geometry>
+    </visual>
+   </link>
+   <joint type="fixed" name="camera_joint">
+        <origin xyz="0.2 0 0" rpy="0 0 0"/>
+        <parent link="chassis"/>
+        <child link="camera"/>
+        <axis xyz="0 1 0"/>
+   </joint>
+<!-- adding Hokuyo sensor -->
+    <link name = 'hokuyo'>
+        <inertial>
+            <mass value ="1e-5"/>
+            <origin xyz="0 0 0" rpy="0 0 0"/>
+            <inertia
+                ixx="1e-6" ixy="0" ixz="0"
+                iyy="1e-6" iyz="0"
+                izz="1e-6"
+            />
+        </inertial>
+        <collision name='hokuyo_collision'>
+            <origin xyz = "0 0 0" rpy="0 0 0"/>
+            <geometry>
+                <box size = "0.1 0.1 0.1"/>
+            </geometry>
+        </collision>
+        <visual name='hokuyo_visual'>
+            <origin xyz = "0 0 0" rpy="0 0 0"/>
+            <geometry>
+                <mesh filename="package://my_robot/meshes/hokuyo.dae"/>
+            </geometry>
+        </visual>
+    </link>
+    <joint type="fixed" name="hokuyo_joint">
+        <origin xyz="0.15 0 0.1" rpy="0 0 0"/>
+        <parent link="chassis"/>
+        <child link="hokuyo"/>
+        <axis xyz = "0 1 0"/>
+    </joint>
+<!-- Changing the color of Left Wheel -->
+    <gazebo reference="left_wheel">
+      <material>Gazebo/Black</material>
+    </gazebo>
+<!-- Changing the color of Right Wheel -->
+    <gazebo reference="right_wheel">
+      <material>Gazebo/Black</material>
+    </gazebo>
+<!-- Changing the color of Chassis -->
+    <gazebo reference="chassis">
+      <material>Gazebo/Orange</material>
+    </gazebo>
+<!-- Changing the color of Camera -->
+    <gazebo reference="camera">
+      <material>Gazebo/Blue</material>
+    </gazebo>
 </robot>
